File: pcb/batt-interface/batt-interface.kicad_pcb (KiCad board)
At the start: 2 copper layers, 33.5 x 14.4 mm, 10 parts, among them IC1 MCP73831T-2ACI_OT, J1 UJC-H-G-SMT-2-P6-TR, J2 Battery, J3 Load

Commit message: Added pull down resistors for CC1 and CC2 to ensure proper charging.
Parts:
- added R3: 5.1k, Resistor_SMD:R_0805_2012Metric_Pad1.20x1.40mm_HandSolder, F.Cu at (130.3, 79.3)
- added R4: 5.1k, Resistor_SMD:R_0805_2012Metric_Pad1.20x1.40mm_HandSolder, F.Cu at (130.3, 69.4)
Routing:
- net unconnected-(J1-CC1-PadA5): track 0.00 -> 16.5 mm
- net unconnected-(J1-CC2-PadB5): track 0.00 -> 16.5 mm
- net GND: track 15.7 -> 25.0 mm
Other:
- board text added: "2026-01-03 v1.1"
- board text removed: "2025-10-26 v1.0"
