File: pcb/batt-interface/batt-interface.kicad_sch (KiCad schematic)
At the start: 12 parts, among them IC1 MCP73831T-2ACI_OT, J1 UJC-H-G-SMT-2-P6-TR, J2 Battery, J3 Load

Commit message: Check in changes to the PCB files. Also checkin main.cpp change to clarify LED colors of status lights
Parts:
- added C3: .1uF, Capacitor_SMD:C_0805_2012Metric_Pad1.18x1.45mm_HandSolder, symbol Device:C
- added IC2: MAX17048G+T10, Garth:SON50P200X200X80-9N-D, symbol Garth Libraries:MAX17048G+T10
- added J4: i2c, Connector_PinHeader_2.54mm:PinHeader_1x04_P2.54mm_Vertical, symbol Connector:Conn_01x04_Socket
Connections:
- net +BATT: now also C3.1, IC2.2 (CELL), IC2.3 (VDD)
- net GND: now also C3.2, IC2.1 (CTG), IC2.4 (GND), IC2.6 (QSTRT), IC2.9 (EP), J4.2 (Pin_2), J4.4 (Pin_4)
- new net SCL: IC2.7 (SCL), J4.3 (Pin_3)
- new net SDA: IC2.8 (SDA), J4.1 (Pin_1)
- no-connect marks 0 -> 1
