File: pcb/pi-shield/pi-shield.kicad_pcb (KiCad board)
At the start: 2 copper layers, 65.5 x 20.1 mm, 9 parts, among them J1 Raspberry_Pi_2_3, J2 LED Header, J3 OLED Display, J4 Rotary Encoder, U1 74AHCT125

Commit message: Several KiCad changes (ngl, not sure what changed here)
Parts:
- added J5: Conn_01x05_Pin, Connector_PinHeader_2.54mm:PinHeader_1x05_P2.54mm_Vertical, F.Cu at (151.7, 82.3)
Connections:
- J1 pad 3: unconnected-(J1-SDA/GPIO2-Pad3) -> /SDA
- J1 pad 5: unconnected-(J1-SCL/GPIO3-Pad5) -> /SCL
- J1 pad 7: unconnected-(J1-GCLK0/GPIO4-Pad7) -> /~ALERT
Routing:
- net /SDA: track 0.00 -> 7.76 mm
- net /SCL: track 0.00 -> 7.76 mm
- net /~ALERT: track 0.00 -> 7.76 mm
- net +5V: track 71.4 -> 75.8 mm
Other:
- board size 65.5 x 20.1 mm -> 65.5 x 23.5 mm
