File: pcb/pi-shield/pi-shield.kicad_sch (KiCad schematic)
At the start: 9 parts, among them J1 Raspberry_Pi_2_3, J2 LED Header, J3 OLED Display, J4 Rotary Encoder, U1 74AHCT125

Commit message: Several KiCad changes (ngl, not sure what changed here)
Parts:
- added J5: Conn_01x05_Pin, Connector_PinHeader_2.54mm:PinHeader_1x05_P2.54mm_Vertical, symbol Connector:Conn_01x05_Pin
Connections:
- net +5V: now also J5.5 (Pin_5)
- net GND: now also J5.1 (Pin_1)
- net SDA: now reaches J1.3 (SDA/GPIO2)
- net SDA: now also J5.4 (Pin_4)
- net SCL: now reaches J1.5 (SCL/GPIO3)
- net SCL: now also J5.3 (Pin_3)
- net ~ALERT: now reaches J1.7 (GCLK0/GPIO4)
- net ~ALERT: now also J5.2 (Pin_2)
- no-connect marks 26 -> 23
